File: SmallSat Peripheral Board/SmallSat Peripheral Board Rev1/Sun_Sensor_Array_Rev1.kicad_sch (KiCad schematic)
At the start: 16 parts

Commit message: ADCS Driver Work
Nothing final yet
Parts:
- R16, R29, R31, R33, R35, R37, R39, R41: renamed from R?; value R -> 3k
- R28, R30, R32, R34, R36, R38, R40, R42: renamed from R?; value R_Photo -> 10k
Connections:
- net 3V3 renamed 5V
