File: SmallSat Peripheral Board/SmallSat Peripheral Board Rev1/ADCS_MCU.kicad_sch (KiCad schematic)
At the start: 0 parts

Commit message: Organized Repository
- Better overall file organization
- Included necessary documentation to be filled out
- Included KiCAD libraries
Parts:
- added C14, C15: 100nF, symbol Device:C
- added C16, C17: 22pF, symbol Device:C
- added R20: 1k, symbol Device:R
- added U7: ATmega328P-P, Package_DIP:DIP-28_W7.62mm, symbol MCU_Microchip_ATmega:ATmega328P-P
- added Y1: 16MHz, symbol Device:Crystal
Connections:
- new net: C16.1, U7.9 (XTAL1/PB6), Y1.2
- new net: R20.1, U7.1 (~{RESET}/PC6)
- new net: C17.1, U7.10 (XTAL2/PB7), Y1.1
- new net: C15.1, U7.20 (AVCC)
- new net: C14.2, U7.21 (AREF)
- new net 5V: C15.2, R20.2, U7.7 (VCC)
- new net COMP_A: U7.23 (PC0)
- new net COMP_B: U7.24 (PC1)
- new net COMP_C: U7.25 (PC2)
- new net CONTROL_PWM: U7.26 (PC3)
- new net GND: C14.1, C16.2, C17.2, U7.22 (GND), U7.8 (GND)
- new net PGM1: U7.17 (PB3)
- new net PGM2: U7.18 (PB4)
- new net PGM3: U7.19 (PB5)
- new net SINK_A: U7.2 (PD0)
- new net SINK_B: U7.3 (PD1)
- new net SINK_C: U7.4 (PD2)
- new net SOURCE_A: U7.5 (PD3)
- new net SOURCE_B: U7.6 (PD4)
- new net SOURCE_C: U7.11 (PD5)
Other:
- note added: "B will be programming port"
- note added: "C will be input port"
- note added: "D will be output port"
- note added: "See pp. 65-71 for port and pin functions"
