File: SmallSat Peripheral Board/SmallSat Peripheral Board Rev1/Crossover_Detectionkicad_sch.kicad_sch (KiCad schematic)
At the start: 0 parts

Commit message: Organized Repository
- Better overall file organization
- Included necessary documentation to be filled out
- Included KiCAD libraries
Parts:
- added C23, C24, C25: 470n, symbol Device:C
- added R47, R48, R49: 1k, symbol Device:R
- added U9: LM339, symbol Comparator:LM339
Connections:
- new net: R47.1, U9.5 (+)
- new net: R49.1, U9.11 (+)
- new net: U9.8 (-), U9.9 (+)
- new net: R48.1, U9.7 (+)
- new net 7.4V: U9.3 (V+)
- new net COMP_A: U9.2
- new net COMP_B: U9.1
- new net COMP_C: U9.13
- new net GND: C23.2, C24.2, C25.2, U9.12 (V-)
- new net Neutral: U9.10 (-), U9.4 (-), U9.6 (-)
- new net Phase A: C23.1, R47.2
- new net Phase B: C24.1, R48.2
- new net Phase C: C25.1, R49.2
