File: SmallSat Peripheral Board/SmallSat Peripheral Board Rev1/MOSFETS.kicad_sch (KiCad schematic)
At the start: 0 parts

Commit message: Organized Repository
- Better overall file organization
- Included necessary documentation to be filled out
- Included KiCAD libraries
Parts:
- added Q1, Q2, Q3, Q4, Q5, Q6: Q_NMOS_GDS, symbol Device:Q_NMOS_GDS
- added R21, R22, R43, R44, R45, R46: 15, symbol Device:R
Connections:
- new net: Q1.1 (G), R21.2
- new net: Q6.1 (G), R46.2
- new net: Q5.1 (G), R45.2
- new net: Q4.1 (G), R44.2
- new net: Q2.1 (G), R22.2
- new net: Q3.1 (G), R43.2
- new net 7.4V: Q1.2 (D), Q3.2 (D), Q5.2 (D)
- new net A_SENSE: Q1.3 (S), Q2.2 (D)
- new net B_SENSE: Q3.3 (S), Q4.2 (D)
- new net C_SENSE: Q5.3 (S), Q6.2 (D)
- new net GND: Q2.3 (S), Q4.3 (S), Q6.3 (S)
- new net HIGH_A: R21.1
- new net HIGH_B: R43.1
- new net HIGH_C: R45.1
- new net LOW_A: R22.1
- new net LOW_B: R44.1
- new net LOW_C: R46.1
Other:
- note added: "Find desirable gate resistors"
