File: SmallSat Peripheral Board/SmallSat Peripheral Board Rev1/MOSFET_Driver.kicad_sch (KiCad schematic)
At the start: 0 parts

Commit message: Organized Repository
- Better overall file organization
- Included necessary documentation to be filled out
- Included KiCAD libraries
Parts:
- added C18: 100nF ceramic, symbol Device:C
- added C19: 400nF, symbol Device:C
- added C20, C21, C22: 50nF, symbol Device:C_Small
- added U8: DRV8300DIPWR, TSSOP_0DIPWR_TEX, symbol SmallSat-Peripherals-Board:DRV8300DIPWR
Connections:
- new net: C21.1, U8.17 (BSTB)
- new net: C22.1, U8.14 (BSTC)
- new net: C20.1, U8.20 (BSTA)
- new net 7.4V: C18.1, C19.1, U8.7 (GVDD)
- new net A_SENSE: C20.2, U8.18 (SHA)
- new net B_SENSE: C21.2, U8.15 (SHB)
- new net C_SENSE: C22.2, U8.12 (SHC)
- new net GND: C18.2, C19.2, U8.8 (GND)
- new net HIGH_A: U8.19 (GHA)
- new net HIGH_B: U8.16 (GHB)
- new net HIGH_C: U8.13 (GHC)
- new net LOW_A: U8.11 (GLA)
- new net LOW_B: U8.10 (GLB)
- new net LOW_C: U8.9 (GLC)
- new net SINK_A: U8.4 (INLA)
- new net SINK_B: U8.5 (INLB)
- new net SINK_C: U8.6 (INLC)
- new net SOURCE_A: U8.1 (INHA)
- new net SOURCE_B: U8.2 (INHB)
- new net SOURCE_C: U8.3 (INHC)
Other:
- note added: "Equivalent capacitance should = 10uF while reducing ESR"
- note added: "See page 19 to calculate bootstrap capacitance"
